Commit message: Optitrack cube

File: home/phd_project/object/cube/cheezit_estimated_object_with_visual_small.urdf (robot description, URDF)
Before this commit: robot cube, 1 links, 0 joints
Links:
- link base_link: geometry visual box size=0.214 0.16 0.061

File: home/phd_project/object/cube/cheezit_object_small.urdf (robot description, URDF)
Before this commit: robot myfirst, 1 links, 0 joints
Links:
- link right_leg: geometry collision box size=0.214 0.16 0.061; visual box size=0.214 0.16 0.061

File: home/phd_project/object/cube/cheezit_particle_no_visual_small.urdf (robot description, URDF)
Before this commit: robot myfirst, 1 links, 0 joints
Links:
- link right_leg: geometry collision box size=0.214 0.16 0.061; visual box size=0.214 0.16 0.061

File: home/phd_project/object/cube/cheezit_particle_with_visual_small.urdf (robot description, URDF)
Before this commit: robot myfirst, 1 links, 0 joints
Links:
- link right_leg: geometry visual box size=0.214 0.16 0.061

File: home/phd_project/object/cube/cheezit_particle_with_visual_small_bl2.urdf (robot description, URDF)
Before this commit: robot myfirst, 1 links, 0 joints
Links:
- link right_leg: geometry visual box size=0.214 0.16 0.061

File: home/phd_project/object/cube/cheezit_real_object_with_visual_small.urdf (robot description, URDF)
Before this commit: robot cube, 1 links, 0 joints
Links:
- link base_link: geometry visual box size=0.214 0.16 0.061

Commit message: cheezit model update

File: home/phd_project/object/cube/cheezit_estimated_object_with_visual_small.urdf (robot description, URDF)
Before this commit: robot cube, 1 links, 0 joints
Links:
- link base_link: geometry visual box size=0.205 0.055 0.165

File: home/phd_project/object/cube/cheezit_object_small.urdf (robot description, URDF)
Before this commit: robot myfirst, 1 links, 0 joints
Links:
- link right_leg: geometry collision box size=0.214 0.061 0.16; visual box size=0.214 0.061 0.16

File: home/phd_project/object/cube/cheezit_particle_no_visual_small.urdf (robot description, URDF)
Before this commit: robot myfirst, 1 links, 0 joints
Links:
- link right_leg: geometry collision box size=0.214 0.061 0.16; visual box size=0.214 0.061 0.16

File: home/phd_project/object/cube/cheezit_particle_with_visual_small.urdf (robot description, URDF)
Before this commit: robot myfirst, 1 links, 0 joints
Links:
- link right_leg: geometry visual box size=0.264 0.066 0.155

File: home/phd_project/object/cube/cheezit_particle_with_visual_small_bl2.urdf (robot description, URDF)
Before this commit: robot myfirst, 1 links, 0 joints
Links:
- link right_leg: geometry visual box size=0.294 0.07 0.15

File: home/phd_project/object/cube/cheezit_real_object_with_visual_small.urdf (robot description, URDF)
Before this commit: robot cube, 1 links, 0 joints
Links:
- link base_link: geometry visual box size=0.2 0.05 0.17
