Commit message: cheezit model update

File: home/phd_project/object/cube/cheezit_est_obj_with_visual_small_PM_hor.urdf (robot description, URDF)
Before this commit: robot myfirst, 1 links, 0 joints
Links:
- removed link right_leg
- added link base_link, mass 0; visual box size=0.16 0.21343700408935547 0.061

File: home/phd_project/object/cube/cheezit_obj_small_hor.urdf (robot description, URDF)
Before this commit: robot myfirst, 1 links, 0 joints
Links:
- link right_leg: geometry collision box size=0.214 0.061 0.16; visual box size=0.16 0.21343700408935547 0.061

File: home/phd_project/object/cube/cheezit_par_no_visual_small_hor.urdf (robot description, URDF)
Before this commit: robot myfirst, 1 links, 0 joints
Links:
- link right_leg: mass 0 -> 1; geometry collision box size=0.214 0.061 0.16; visual box size=0.16 0.21343700408935547 0.061

File: home/phd_project/object/cube/cheezit_par_with_visual_small_PE_hor.urdf (robot description, URDF)
Before this commit: robot cube, 1 links, 0 joints
Links:
- removed link base_link
- added link right_leg, mass 0; visual box size=0.145 0.23343700408935547 0.08

File: home/phd_project/object/cube/cheezit_par_with_visual_small_PM_hor.urdf (robot description, URDF)
Before this commit: robot myfirst, 1 links, 0 joints
Links:
- link right_leg: mass 1 -> 0; geometry visual box size=0.13 0.250 0.09

File: home/phd_project/object/cube/cheezit_real_obj_with_visual_small_hor.urdf (robot description, URDF)
Before this commit: robot cube, 1 links, 0 joints
Links:
- link base_link: geometry visual box size=0.18 0.2 0.05
