Commit message: correct the rotation

File: home/phd_project/object/cube/cheezit_obj_small_hor.urdf (robot description, URDF)
Before this commit: robot myfirst, 1 links, 0 joints
Links:
- link right_leg: geometry collision box size=0.16 0.21343700408935547 0.061; visual box size=0.16 0.21343700408935547 0.061

File: home/phd_project/object/cube/cheezit_par_no_visual_small_hor.urdf (robot description, URDF)
Before this commit: robot myfirst, 1 links, 0 joints
Links:
- link right_leg: geometry collision box size=0.16 0.21343700408935547 0.061; visual box size=0.16 0.21343700408935547 0.061
