Commit message: code update

File: home/phd_project/object/cube/base_of_cheezit.urdf (robot description, URDF)
Before this commit: robot myfirst, 1 links, 0 joints
Links:
- link right_leg: geometry collision box size=0.207 0.2185 0.1006; visual box size=0.207 0.2185 0.1006

Commit message: code update

File: home/phd_project/object/cube/base_of_cheezit.urdf (robot description, URDF)
Before this commit: robot myfirst, 1 links, 0 joints
Links:
- link right_leg: geometry collision box size=0.207 0.2185 0.1681; visual box size=0.207 0.2185 0.1681
