Commit message: code update

File: home/phd_project/object/cylinder_particle_no_visual_small.urdf (robot description, URDF)
Before this commit: robot myfirst, 1 links, 0 joints
Links:
- link base_link: geometry collision cylinder length=10.185500144958496 radius=3.3829689025878906; visual cylinder length=10.185500144958496 radius=3.3829689025878906
