Commit message: code update

File: home/phd_project/object/soup/camsoup_dope_obj_with_visual_small_PE_hor.urdf (robot description, URDF)
Before this commit: robot cube, 1 links, 0 joints
Links:
- link base_link: geometry visual cylinder length=10.00 radius=3.3829689025878906

File: home/phd_project/object/soup/camsoup_est_obj_with_visual_small_PE_hor.urdf (robot description, URDF)
Before this commit: robot cube, 1 links, 0 joints
Links:
- link base_link: geometry visual cylinder length=10.00 radius=3.3829689025878906

File: home/phd_project/object/soup/camsoup_est_obj_with_visual_small_PM_hor.urdf (robot description, URDF)
Before this commit: robot cube, 1 links, 0 joints
Links:
- link base_link: geometry visual cylinder length=10.00 radius=3.3829689025878906

File: home/phd_project/object/soup/camsoup_obj_small_hor.urdf (robot description, URDF)
Before this commit: robot myfirst, 1 links, 0 joints
Links:
- link obj_in_sim: geometry collision cylinder length=10.00 radius=3.3829689025878906; visual cylinder length=10.00 radius=3.3829689025878906

File: home/phd_project/object/soup/camsoup_par_no_visual_small_hor.urdf (robot description, URDF)
Before this commit: robot myfirst, 1 links, 0 joints
Links:
- link right_leg: geometry collision cylinder length=10.00 radius=3.3829689025878906; visual cylinder length=10.00 radius=3.3829689025878906

File: home/phd_project/object/soup/camsoup_real_obj_with_visual_small_hor.urdf (robot description, URDF)
Before this commit: robot cube, 1 links, 0 joints
Links:
- link base_link: geometry visual cylinder length=10.00 radius=3.3829689025878906
