Commit message: code and urdf update

File: home/project/object/soup/soup_contact_test_obj_hor.urdf (robot description, URDF)
Before this commit: robot myfirst, 1 links, 0 joints
Links:
- link obj_in_sim: geometry collision cylinder length=0.1000 radius=0.033829689025878906; visual cylinder length=0.0800 radius=0.013829689025878906
