Commit message: change name

File: home/project/object/cracker/cracker_contact_test_obj_hor.urdf (robot description, URDF)
Before this commit: robot myfirst, 1 links, 0 joints
Links:
- link right_leg: geometry collision box size=0.16 0.21343700408935547 0.061; visual box size=0.14 0.19343700408935547 0.041

File: home/project/object/soup/soup_real_obj_hor.urdf (robot description, URDF)
Before this commit: robot myfirst, 1 links, 0 joints
Links:
- removed link right_leg
- added link obj_in_sim, mass 1; collision cylinder length=0.1000 radius=0.033829689025878906; visual cylinder length=0.1000 radius=0.033829689025878906
