Commit message: code and urdf update

File: home/project/object/cracker/cracker_par_with_visual_CV_hor.urdf (robot description, URDF)
Before this commit: robot myfirst, 1 links, 0 joints
Links:
- link right_leg: geometry visual box size=0.16 0.21343700408935547 0.061

File: home/project/object/cracker/cracker_par_with_visual_PB_hor.urdf (robot description, URDF)
Before this commit: robot myfirst, 1 links, 0 joints
Links:
- link right_leg: geometry visual box size=0.16 0.21343700408935547 0.061

File: home/project/object/soup/soup_par_with_visual_CV_hor.urdf (robot description, URDF)
Before this commit: robot myfirst, 1 links, 0 joints
Links:
- link right_leg: geometry visual cylinder length=0.1000 radius=0.033829689025878906

File: home/project/object/soup/soup_par_with_visual_PB_hor.urdf (robot description, URDF)
Before this commit: robot myfirst, 1 links, 0 joints
Links:
- link right_leg: geometry visual cylinder length=0.1000 radius=0.033829689025878906
