Commit message: code update

File: home/project/object/cracker/cracker_real_obj_with_visual_hor.urdf (robot description, URDF)
Before this commit: robot cube, 1 links, 0 joints
Links:
- link base_link: geometry visual box size=0.26 0.21343700408935547 0.062

Commit message: code update

File: home/project/object/cracker/cracker_real_obj_with_visual_hor.urdf (robot description, URDF)
Before this commit: robot cube, 1 links, 0 joints
Links:
- link base_link: geometry visual box size=0.2600016 0.21343700408935547 0.062

File: home/project/object/soup/soup_real_obj_with_visual_hor.urdf (robot description, URDF)
Before this commit: robot cube, 1 links, 0 joints
Links:
- link base_link: geometry visual cylinder length=0.260001 radius=0.033829689025878906
