Commit message: model update

File: home/project/object/cracker/cracker_par_with_visual_PB_hor.urdf (robot description, URDF)
Before this commit: robot myfirst, 1 links, 0 joints
Links:
- removed link right_leg
- added link cracker, mass 0; visual mesh filename=textured_simple_reoriented.obj scale=1 1 1
- added link fake; visual box size=0.0001 0.0001 0.0001
Joints:
- added joint fake_2_cracker: type fixed, parent fake, child cracker, origin xyz=0.0 0.0 0.0 rpy=0.0 -1.5707963 1.5707963

Commit message: code update

File: home/project/object/cracker/cracker_par_with_visual_PB_hor.urdf (robot description, URDF)
Before this commit: robot myfirst, 2 links, 1 joints
Links:
- removed link fake
Joints:
- removed joint fake_2_cracker

File: home/project/object/soup/soup_par_with_visual_PB_hor.urdf (robot description, URDF)
Before this commit: robot myfirst, 1 links, 0 joints
Links:
- removed link right_leg
- added link soup, mass 0; visual mesh filename=textured_simple_reoriented.obj scale=1 1 1

Commit message: code update

File: home/project/object/cracker/cracker_par_with_visual_PB_hor.urdf (robot description, URDF)
Before this commit: robot myfirst, 1 links, 0 joints
Links:
- link cracker: geometry visual box size=0.16 0.21343700408935547 0.061
