Commit message: new model

File: home/project/object/others/shelves.urdf (robot description, URDF)
Before this commit: robot myfirst, 1 links, 0 joints
Links:
- removed link right_leg
- added link back, mass 0.75; collision box size=0.6915 0.694 0.019; visual box size=0.6915 0.694 0.019
- added link bottom, mass 0.75; collision box size=0.33 0.7285 0.019; visual box size=0.33 0.7285 0.019
- added link left, mass 0.75; collision box size=0.33 0.694 0.0185; visual box size=0.33 0.694 0.0185
- added link middle, mass 0.75; collision box size=0.301 0.6915 0.018; visual box size=0.301 0.6915 0.018
- added link right, mass 0.75; collision box size=0.33 0.694 0.0185; visual box size=0.33 0.694 0.0185
Joints:
- added joint back_to_bottom: type fixed, parent back, child bottom, origin xyz=-0.1555 -0.0 -0.3565
- added joint back_to_left: type fixed, parent back, child left, origin xyz=-0.1555 0.355 0
- added joint back_to_middle: type fixed, parent back, child middle, origin xyz=-0.16 -0.0 0.06
- added joint back_to_right: type fixed, parent back, child right, origin xyz=-0.1555 -0.355 0

Commit message: new model

File: home/project/object/others/shelves.urdf (robot description, URDF)
Before this commit: robot myfirst, 5 links, 4 joints
Links:
- added link top, mass 0.75; collision box size=0.33 0.7285 0.019; visual box size=0.33 0.7285 0.019
Joints:
- added joint back_to_top: type fixed, parent back, child top, origin xyz=-0.1555 -0.0 0.3565
