Commit message: update model

File: home/project/object/others/table.urdf (robot description, URDF)
Before this commit: robot base_box, 5 links, 4 joints
Links:
- link back_short: mass None -> 0.75
- link base_link: mass None -> 0.75
- link forward_short: mass None -> 0.75
- link left_long: mass None -> 0.75
- link right_long: mass None -> 0.75

Commit message: new model

File: home/project/object/others/table.urdf (robot description, URDF)
Before this commit: robot base_box, 5 links, 4 joints
Links:
- link base_link: geometry collision box size=1.20 1.20 0.016; visual box size=1.20 1.20 0.016
