Commit message: code and model update

File: home/project/object/Ketchup/Ketchup_contact_test_obj_hor.urdf (robot description, URDF)
Before this commit: robot myfirst, 2 links, 1 joints
Links:
- removed link fake
- link Ketchup: mass 0 -> 0.5
Joints:
- removed joint fake_2_Ketchup

File: home/project/object/Ketchup/Ketchup_est_obj_with_visual_CV_hor.urdf (robot description, URDF)
Before this commit: robot myfirst, 2 links, 1 joints
Links:
- removed link fake
- link Ketchup: mass 0 -> 0.5
Joints:
- removed joint fake_2_Ketchup

File: home/project/object/Ketchup/Ketchup_est_obj_with_visual_PB_hor.urdf (robot description, URDF)
Before this commit: robot myfirst, 2 links, 1 joints
Links:
- removed link fake
- link Ketchup: mass 0 -> 0.5
Joints:
- removed joint fake_2_Ketchup

File: home/project/object/Ketchup/Ketchup_par_no_visual_hor.urdf (robot description, URDF)
Before this commit: robot myfirst, 2 links, 1 joints
Links:
- removed link fake
- link Ketchup: mass 0 -> 0.5
Joints:
- removed joint fake_2_Ketchup

File: home/project/object/Ketchup/Ketchup_par_with_visual_PB_hor.urdf (robot description, URDF)
Before this commit: robot myfirst, 2 links, 1 joints
Links:
- removed link fake
- link Ketchup: mass 0 -> 0.5
Joints:
- removed joint fake_2_Ketchup

File: home/project/object/OrangeJuice/OrangeJuice_contact_test_obj_hor.urdf (robot description, URDF)
Before this commit: robot object, 2 links, 1 joints
Links:
- removed link fake
Joints:
- removed joint fake_2_OrangeJuice

File: home/project/object/OrangeJuice/OrangeJuice_est_obj_with_visual_CV_hor.urdf (robot description, URDF)
Before this commit: robot object, 2 links, 1 joints
Links:
- removed link fake
Joints:
- removed joint fake_2_OrangeJuice

File: home/project/object/OrangeJuice/OrangeJuice_est_obj_with_visual_PB_hor.urdf (robot description, URDF)
Before this commit: robot object, 2 links, 1 joints
Links:
- removed link fake
Joints:
- removed joint fake_2_OrangeJuice

File: home/project/object/OrangeJuice/OrangeJuice_par_no_visual_hor.urdf (robot description, URDF)
Before this commit: robot object, 2 links, 1 joints
Links:
- removed link fake
Joints:
- removed joint fake_2_OrangeJuice

File: home/project/object/OrangeJuice/OrangeJuice_par_with_visual_CV_hor.urdf (robot description, URDF)
Before this commit: robot object, 2 links, 1 joints
Links:
- removed link fake
Joints:
- removed joint fake_2_OrangeJuice

Commit message: code update

File: home/project/object/Ketchup/Ketchup_contact_test_obj_hor.urdf (robot description, URDF)
Before this commit: robot myfirst, 1 links, 0 joints
Links:
- link Ketchup: geometry collision mesh filename=Ketchup.obj scale=1 1 1; visual mesh filename=Ketchup_sim.obj scale=0.5 0.5 0.5

File: home/project/object/Ketchup/Ketchup_est_obj_with_visual_CV_hor.urdf (robot description, URDF)
Before this commit: robot myfirst, 1 links, 0 joints
Links:
- link Ketchup: geometry visual mesh filename=Ketchup_sim.obj scale=1 1 1

File: home/project/object/Ketchup/Ketchup_est_obj_with_visual_PB_hor.urdf (robot description, URDF)
Before this commit: robot myfirst, 1 links, 0 joints
Links:
- link Ketchup: geometry visual mesh filename=Ketchup_sim.obj scale=1 1 1

File: home/project/object/Ketchup/Ketchup_par_no_visual_hor.urdf (robot description, URDF)
Before this commit: robot myfirst, 1 links, 0 joints
Links:
- link Ketchup: geometry collision mesh filename=Ketchup.obj scale=1 1 1; visual mesh filename=Ketchup_sim.obj scale=1 1 1

File: home/project/object/Ketchup/Ketchup_par_with_visual_PB_hor.urdf (robot description, URDF)
Before this commit: robot myfirst, 1 links, 0 joints
Links:
- link Ketchup: geometry visual mesh filename=Ketchup_sim.obj scale=1 1 1
