Commit message: code update

File: home/project/data/bullet3-master/examples/pybullet/gym/pybullet_data/franka_panda/panda_pump.urdf (robot description, URDF)
Before this commit: robot panda, 13 links, 12 joints
Links:
- removed link panda_grasptarget
- removed link panda_hand
- removed link panda_leftfinger
- removed link panda_rightfinger
- added link extention_stick, mass 1; collision cylinder length=0.178 radius=0.0125; visual cylinder length=0.178 radius=0.0125
- added link pump, mass .81; collision mesh filename=package://meshes/collision/pump.obj; visual mesh filename=package://meshes/visual/pump.obj
- added link pump_camera_holder, mass .81; collision mesh filename=package://meshes/collision/pump_camera_holder.obj; visual mesh filename=package://meshes/visual/pump_camera_holder.obj
Joints:
- removed joint panda_finger_joint1
- removed joint panda_finger_joint2
- removed joint panda_grasptarget_hand
- added joint pump_camera_holder_joint1: type fixed, parent pump, child pump_camera_holder, origin xyz=0 0 0.0 rpy=0.1 1.5707963 0
- added joint pump_extention_stick: type fixed, parent pump, child extention_stick, origin xyz=0 -0.177655 0 rpy=0 0 0
- joint panda_hand_joint: child panda_hand -> pump; origin xyz=0 0 0 rpy=0 0 -0.785398163397 -> xyz=0 0 0 rpy=-1.5707963 0 2.3561944366

Commit message: code update

File: home/project/data/bullet3-master/examples/pybullet/gym/pybullet_data/franka_panda/panda_pump.urdf (robot description, URDF)
Before this commit: robot panda, 12 links, 11 joints
Links:
- added link panda_pumptarget, mass 0.0
Joints:
- removed joint panda_hand_joint
- added joint extention_stick_pumptarget: type fixed, parent extention_stick, child panda_pumptarget, origin xyz=0 0 0.0 rpy=0 0 0
- added joint panda_pump_joint: type fixed, parent panda_link8, child pump, origin xyz=0 0 0 rpy=-1.5707963 0 2.3561944366
