Commit message: code update

File: home/project/object/Parmesan/Parmesan_real_obj_with_visual_hor.urdf (robot description, URDF)
Before this commit: robot myfirst, 1 links, 0 joints
Links:
- link Parmesan: geometry visual mesh filename=Parmesan.obj scale=1.2 1 1

File: home/project/object/soup/soup_obse_obj_with_visual_hor.urdf (robot description, URDF)
Before this commit: robot cube, 1 links, 0 joints
Links:
- link base_link: geometry visual cylinder length=0.1000 radius=0.033829689025878906

File: home/project/object/soup/soup_real_obj_with_visual_hor.urdf (robot description, URDF)
Before this commit: robot cube, 1 links, 0 joints
Links:
- link base_link: geometry visual cylinder length=0.1100 radius=0.033829689025878906
